File: IoT12.kicad_pcb (KiCad board)
At the start: 2 copper layers, 99.1 x 69.8 mm, 103 parts, among them J10 USB_B_Micro, J11 Conn_ARM_JTAG_SWD_10, Q1 MMBT2222, Q2 MMBT2222, Q3 AOD403, SW1 Rotary encoder EC11 Plum 15mm, SW2 SW_Push, U1 ATSAMD21G, U2 ADS1115IDGS, U3 INA826AID, U4 INA826AID, U5 LM2596S-ADJ, Y1 32768Hz

Commit message: V2.0 pcb.
Parts:
- removed C72: 100uF/35V, Capacitor_SMD:CP_Elec_6.3x7.7
- removed NT2: ~, NetTie-extra:NetTie-2_SMD_Pad0.25mm
- added C22: 1nF, Capacitor_SMD:C_0805_2012Metric_Pad1.18x1.45mm_HandSolder, F.Cu at (-44.5, 15.2)
- added J9: Conn_ARM_JTAG_SWD_10, Connector_PinHeader_2.54mm:PinHeader_2x05_P2.54mm_Vertical, B.Cu at (14.0, -39.4)
- added R84: 1M, Resistor_SMD:R_0805_2012Metric_Pad1.20x1.40mm_HandSolder, F.Cu at (-47.0, 15.2)
- added REF**: OSHW-Logo_19x20mm_SilkScreen, Symbol:OSHW-Logo_19x20mm_SilkScreen, B.Cu at (34.2, -10.3)
- added TP1: TestPoint, TestPoint-extra:TestPoint_Pad_D0.75mm, F.Cu at (-36.8, -26.7)
- added TP2: TestPoint, TestPoint-extra:TestPoint_Pad_D0.75mm, F.Cu at (-36.8, -25.4)
- added TP3: TestPoint, TestPoint-extra:TestPoint_Pad_D0.75mm, F.Cu at (-36.8, -24.1)
- added TP4: TestPoint, TestPoint-extra:TestPoint_Pad_D0.75mm, F.Cu at (-36.8, -22.9)
- added U6: AT24C32, Package_SO:SO-8_3.9x4.9mm_P1.27mm, F.Cu at (-37.5, -16.5)
- F1, F2: moved to B.Cu
- moved F1 1.20 mm to (41.9, 12.7)
- moved F2 0.90 mm to (45.7, 5.08)
Connections:
- net IRON_POWER renamed IRON_CURRENT
- A1 pad 12: HEAT_INT -> Net-(A1-Pad12)
- A1 pad 2: ESP32_EN -> EN
- A1 pad 25: ESP32_IO0 -> Net-(A1-Pad25)
- A1 pad 34: ESP32_RXD -> Net-(A1-Pad34)
- A1 pad 35: ESP32_TXD -> Net-(A1-Pad35)
- A1 pad 6: Net-(A1-Pad6) -> HEAT_INT
- J10 pad 5: Net-(J10-Pad5) -> GND
- J10 pad 6: Net-(J10-Pad5) -> Net-(C22-Pad1)
- U1 pad 12: Net-(U1-Pad12) -> /Brain/D9
- U1 pad 15: ESP32_RXD -> /Brain/D1
- U1 pad 16: ESP32_TXD -> /Brain/D0
- U1 pad 27: ESP32_EN -> /Brain/D10
- U1 pad 28: ESP32_IO0 -> Net-(U1-Pad28)
Routing:
- net EN: track 0.00 -> 72.1 mm
- net Net-(A1-Pad23): track 0.00 -> 49.1 mm, vias 0 -> 2
- net Net-(A1-Pad13): track 0.00 -> 42.6 mm, vias 0 -> 1
- net Net-(A1-Pad12): track 0.00 -> 34.5 mm, vias 0 -> 1
- net ESP32_TXD: track 33.3 -> 0.00 mm, vias 2 -> 0
- net ESP32_EN: track 31.8 -> 0.00 mm, vias 2 -> 0
- net ESP32_RXD: track 30.2 -> 0.00 mm, vias 2 -> 0
- net Net-(A1-Pad15): track 0.00 -> 29.4 mm, vias 0 -> 1
- net ESP32_IO0: track 27.0 -> 0.00 mm, vias 2 -> 0
- net /Brain/D0: track 0.00 -> 26.1 mm, vias 0 -> 2
- net /Brain/D9: track 0.00 -> 25.0 mm, vias 0 -> 2
- net /Brain/D10: track 0.00 -> 24.6 mm, vias 0 -> 2
- net /Brain/D1: track 0.00 -> 22.9 mm, vias 0 -> 2
- net HEAT_INT: track 19.6 -> 38.7 mm, vias 2 -> 4
- net Net-(C22-Pad1): track 0.00 -> 18.1 mm
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Other:
- board text added: "1, blue, shake"
- board text added: "2, white, NTC"
- board text added: "24V max"
- board text added: "3, green, ESD"
- board text added: "4, black, T12-"
- board text added: "5, red, T12+"
- board text added: "D0"
- board text added: "D1"
- board text added: "D10"
- board text added: "D9"
- board text added: "IoT12, 2021-02-22, V2.0 https://atoomnet.net"
- board text added: "JTAG ESP32"
- board text added: "Power supply suggestions: 12V@1.5A (18W) 15V@1.9A (28W) 19V@2.4A (45W) 24V@3.0A (72W)"
- board text added: "Q: If the Continuum's told you once, they've told you a thousand times. DON'T - PROVOKE - THE BORG!!"
- board text added: "https://github.com/atoomnetmarc/IoT12-hardware License: Creative Commons Attribution-NonCommercial 3.0 Unported"
- board text removed: "24V"
- board text removed: "IoT12, 2021-02-21, V2.0 https://atoomnet.net"
