File: Output.sch (KiCad schematic (older format))
At the start: 37 parts, among them Q1 2N7002, Q2 2N7002, Q3 AOD403, U6 LM393, U7 74HC125

Commit message: V2.0 pcb.
Parts:
- removed C12, C17, C18: 100nF, Capacitor_SMD:C_0805_2012Metric_Pad1.18x1.45mm_HandSolder, symbol Device:C
- removed C14: 10uF, Capacitor_SMD:C_0805_2012Metric_Pad1.18x1.45mm_HandSolder, symbol Device:C
- removed D2: BAV99, Package_TO_SOT_SMD:SOT-23, symbol Diode:BAV99
- removed Q1: 2N7002, Package_TO_SOT_SMD:SOT-23, symbol Transistor_FET:2N7002
- removed R22, R45: 10k, Resistor_SMD:R_0805_2012Metric_Pad1.20x1.40mm_HandSolder, symbol Device:R
- removed R33, R34, R35, R42: 100k, Resistor_SMD:R_0805_2012Metric_Pad1.20x1.40mm_HandSolder, symbol Device:R
- removed R44: 39k, Resistor_SMD:R_0805_2012Metric_Pad1.20x1.40mm_HandSolder, symbol Device:R
- removed R9: 1k, Resistor_SMD:R_0805_2012Metric_Pad1.20x1.40mm_HandSolder, symbol Device:R
- removed U6: LM393, Package_SO:SO-8_3.9x4.9mm_P1.27mm, symbol Comparator:LM393
- removed U7: 74HC125, Package_SO:SOIC-14_3.9x8.7mm_P1.27mm, symbol 74xx:74LS125
- added A3: max98357, Module-extra:max98357, symbol Module-extra:max98357
- added Q1: MMBT2222, Package_TO_SOT_SMD:SOT-23, symbol Transistor_BJT:BC817
- added R72: 100k, Resistor_SMD:R_0805_2012Metric_Pad1.20x1.40mm_HandSolder, symbol Device:R
- Q2: value 2N7002 -> MMBT2222; symbol Transistor_FET:2N7002 -> Transistor_BJT:BC817
- R32: value 100k -> 1k
- R34: renamed from R7; value 100R -> 1k
- renumbered D1 to D11, D4 to D5, D7 to D8, D3 to D9, J108 to J3, J109 to J4, J107 to J5, NT2 to NT4, NT3 to NT5, R13 to R33, R21 to R58, R19 to R59, R36 to R71, R39 to R82, R40 to R83
Connections:
- net ~ENABLE~_OVERTEMPERATURE is gone; now on net PWM_HEAT: R34.2, R59.1, R71.1
- net +5V: now also A3.7 (VCC)
- net GND: now also A3.6 (GND), Q1.2 (E); no longer R32.2
- net LCD_LED: now also R32.2; no longer R32.1
- net GATE: now reaches D9.2 (A), Q3.1 (G), R33.1, R58.2
- net at A2.7 (~LED): now also Q1.3 (C)
- net SAFE_PWM_HEAT: no longer names the net of Q2.1 (B), R34.1
- new net: Q1.1 (B), R32.1
- new net I2S_BCK: A3.2 (BLCK)
- new net I2S_DATA: A3.3 (DIN)
- new net I2S_GAIN0: A3.4 (GAIN), R72.1
- new net I2S_GAIN1: R72.2
- new net I2S_SD: A3.5 (SD)
- new net I2S_WS: A3.1 (LRC)
- no-connect marks 1 -> 2
Other:
- note added: "Bleep bloop module"
- note removed: "About 0.5s timeout \nafter PWM fail \n(equal to 100% dutycycle) \nto switch off output."
- note removed: "Block heating when TEMP reaches 0.96V or 520°C (above ambient).\n\n"
- note removed: "Heater PWM failsafe"
- note removed: "Heater overheat failsafe"
- moved on the sheet: A2, D11, D5, D8, D9, NT4, NT5, Q3, R1, R33, R34, R58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
