File: Control Board/IoT12 Control Board.sch (KiCad schematic (older format))
At the start: 4 parts

Commit message: Updated revision date.
Changed lines of the file:
@@
 Sheet 1 5
 Title "IoT12-hardware"
-Date "2021-03-13"
+Date "2021-03-27"
 Rev "V2.1"
 Comp ""
@@
 $EndComp
 $Sheet
-S 1550 600  900  800
+S 550  1650 900  800
 U 6029EF83
 F0 "Input" 50
@@
 $EndSheet
 $Sheet
-S 2550 600  900  800
+S 550  2700 900  800
 U 60488463
 F0 "Brain" 50
@@
 $EndSheet
 $Sheet
-S 3550 600  900  800
+S 550  3750 900  800
 U 604A18A1
 F0 "Output" 50
